File: SolenoidBreakout/SolenoidBreakout.sch (KiCad schematic (older format))
At the start: 16 parts, among them J1 Conn_01x02, J2 949, J3 MiniFitPower, Q1 Q_NPN_EBC, U1 IRFZ44N

Commit message: Adding servo firmware
Parts:
- S1: symbol dk_Tactile-Switches:1825910-7 -> SolenoidBreakout-rescue:1825910-7-dk_Tactile-Switches
Changed lines of the file:
@@
 EESchema Schematic File Version 4
-LIBS:SolenoidBreakout-cache
 EELAYER 30 0
 EELAYER END
@@
 $EndComp
 $Comp
-L dk_Tactile-Switches:1825910-7 S1
+L SolenoidBreakout-rescue:1825910-7-dk_Tactile-Switches S1
 U 1 1 5EC7000A
 P 2800 3600
